File: RZIT_LF-01_Schematics/RZIT_LF-01/back_plate.kicad_sch (KiCad schematic)
At the start: 0 parts

Commit message: small changes
Parts:
- added J?: 52437-2471, 524372471, symbol SamacSys_Parts:52437-2471
- added J?: Conn_01x02, symbol Connector_Generic:Conn_01x02
Connections:
- new net +7.5V: J?.1 (Pin_1), J?.2, J?.3
- new net DET_01: J?.7
- new net DET_02: J?.8
- new net DET_03: J?.9
- new net DET_04: J?.10
- new net DET_05: J?.11
- new net DET_06: J?.12
- new net DET_07: J?.13
- new net DET_08: J?.14
- new net DET_09: J?.15
- new net DET_10: J?.16
- new net DET_11: J?.17
- new net DET_12: J?.18
- new net GND: J?.1, J?.2 (Pin_2), J?.4
- new net TOF_INT: J?.20
- new net TOF_SCL: J?.22
- new net TOF_SDA: J?.21
- new net TOF_XSHUT: J?.23
- no-connect marks 0 -> 9

Commit message: as5600 cos
Parts:
- added IC?: AS5600-ASOM, SOIC127P600X175-8N, symbol SamacSys_Parts:AS5600-ASOM
- J?: footprint (none) -> Connector_JST:JST_XH_B2B-XH-AM_1x02_P2.50mm_Vertical
Connections:
- no-connect marks 9 -> 8
Changed lines of the file:
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@@
   (no_connect (at 63.5 193.04))
   (no_connect (at 45.72 158.75))
-  (no_connect (at 63.5 149.86))
   (no_connect (at 60.96 193.04))
   (wire (pts (xy 53.34 158.75) (xy 53.34 165.1))
@@
       (effects (font (size 1.27 1.27)) (justify left))
     )
-    (property "Footprint" "" (id 2) (at 133.35 176.53 0)
+    (property "Footprint" "Connector_JST:JST_XH_B2B-XH-AM_1x02_P2.50mm_Vertical" (id 2) (at 133.35 176.53 0)
       (effects (font (size 1.27 1.27)) hide)
     )
@@
     (pin "1")
   )
+  (symbol (lib_id "SamacSys_Parts:AS5600-ASOM") (at 247.65 146.05 0) (unit 1)
+    (in_bom yes) (on_board yes) (fields_autoplaced)
+    (property "Reference" "IC?" (id 0) (at 262.89 138.43 0))
+    (property "Value" "AS5600-ASOM" (id 1) (at 262.89 140.97 0))
+    (property "Footprint" "SOIC127P600X175-8N" (id 2) (at 274.32 143.51 0)
+      (effects (font (size 1.27 1.27)) (justify left) hide)
+    )
+    (property "Datasheet" "https://datasheet.datasheetarchive.com/originals/distributors/DKDS-11/214624.pdf" (id 3) (at 274.32 146.05 0)
+      (effects (font (size 1.27 1.27)) (justify left) hide)
+    )
+    (property "Description" "IC SENSOR MAG ROTARY 12BIT 8SOIC" (id 4) (at 274.32 148.59 0)
+      (effects (font (size 1.27 1.27)) (justify left) hide)
+    )
+    (property "Height" "1.75" (id 5) (at 274.32 151.13 0)
+      (effects (font (size 1.27 1.27)) (justify left) hide)
+    )
+    (property "Mouser Part Number" "985-AS5600-ASOM" (id 6) (at 274.32 153.67 0)
+      (effects (font (size 1.27 1.27)) (justify left) hide)
+    )
+    (property "Mouser Price/Stock" "https://www.mouser.co.uk/ProductDetail/ams/AS5600-ASOM?qs=KTMMzrZdriG6aU1h9lJCUQ%3D%3D" (id 7) (at 274.32 156.21 0)
+      (effects (font (size 1.27 1.27)) (justify left) hide)
+    )
+    (property "Manufacturer_Name" "ams" (id 8) (at 274.32 158.75 0)
+      (effects (font (size 1.27 1.27)) (justify left) hide)
+    )
+    (property "Manufacturer_Part_Number" "AS5600-ASOM" (id 9) (at 274.32 161.29 0)
+      (effects (font (size 1.27 1.27)) (justify left) hide)
+    )
+    (pin "1")
+    (pin "2")
+    (pin "3")
+    (pin "4")
+    (pin "5")
+    (pin "6")
+    (pin "7")
+    (pin "8")
+  )
 )
