File: RZIT_LF-01_Schematics/RZIT_LF-01/front_plate.kicad_sch (KiCad schematic)
At the start: 37 parts

Commit message: Changes
addetd
Parts:
- removed U?: VL53L1CXV0FY1, Sensor_Distance:ST_VL53L1x, symbol Sensor_Distance:VL53L1CXV0FY1
- added C?: 100nF, symbol Device:C
- added C?: 4.7uF, symbol Device:C
- added R? (x4): 10k, symbol Device:R
- added U?: VL53L1CXV0FY1, Sensor_Distance:ST_VL53L1x, symbol Sensor_Distance:VL53L1CXV0FY1
Connections:
- net +3V3: now also C?.1, C?.1, R?.1, R?.1, R?.1, R?.1, U?.1 (AVDDVCSEL), U?.11 (AVDD)
- net GND: now also C?.2, C?.2, U?.12 (GND), U?.2 (AVSSVCSEL), U?.3 (GND), U?.4 (GND), U?.6 (GND)
- net GPIO: now reaches R?.2, U?.3
- new net TOF_INT: R?.2, U?.7 (GPIO1)
- new net TOF_SCL: R?.2, U?.10 (SCL)
- new net TOF_SDA: R?.2, U?.9 (SDA)
- new net TOF_XSHUT: R?.2, U?.5 (XSHUT)

Commit message: schematic update
schematic update
Parts:
- added C? (x2): 10uF, symbol Device:C
- added D?: LED, symbol Device:LED
- added J?: 52437-2471, 524372471, symbol SamacSys_Parts:52437-2471
- added R?: 200, symbol Device:R
- added U?: AMS1117-3.3, Package_TO_SOT_SMD:SOT-223-3_TabPin2, symbol Regulator_Linear:AMS1117-3.3
Connections:
- net +3V3: now also C?.1, R?.1, U?.2 (VO)
- net GND: now also C?.2, C?.2, D?.1 (K), U?.1 (GND)
- net DET_05: now reaches R?.2, U?.3
- net DET_03: now reaches R?.2, U?.3
- net DET_06: now reaches R?.2, U?.3
- net DET_02: now reaches R?.2, U?.3
- net DET_07: now reaches R?.2, U?.3
- net DET_09: now reaches R?.2, U?.3
- net DET_12: now reaches R?.2, U?.3
- net DET_01: now reaches R?.2, U?.3
- net DET_11: now reaches R?.2, U?.3
- net DET_08: now reaches R?.2, U?.3
- net DET_10: now reaches R?.2, U?.3
- net GPIO renamed DET_04
- new net: D?.2 (A), R?.2
- new net +7.5V: C?.1, U?.3 (VI)

Commit message: small changes
Connections:
- net +7.5V: now also J?.2, J?.3
- net DET_01: now also J?.7
- net DET_02: now also J?.8
- net DET_03: now also J?.9
- net DET_04: now also J?.10
- net DET_05: now also J?.11
- net DET_06: now also J?.12
- net DET_07: now also J?.13
- net DET_08: now also J?.14
- net DET_09: now also J?.15
- net DET_10: now also J?.16
- net DET_11: now also J?.17
- net DET_12: now also J?.18
- net GND: now also J?.1, J?.4
- net TOF_INT: now also J?.20
- net TOF_SCL: now also J?.22
- net TOF_SDA: now also J?.21
- net TOF_XSHUT: now also J?.23
- no-connect marks 0 -> 9
